File: design/pcb/ventmon_t0.3.brd (EAGLE design)
At the start: 85 x 56 mm, 74 parts, among them IC1 BME280BM280-HAT, J4 MJ-3536N, J6 Header-16, J7 Header-12, U1 W5500, U2 ADS1115IDGST, Y1 25MHz

Commit message: fixed 5V to flow sensor
Connections:
- removed net VPOE: J1.1, J7.3
- new net +5V: FLOWSENSOR.2, J1.1, J7.3
- net +3V3: no longer FLOWSENSOR.2
Routing:
- net +5V: track 0.00 -> 84.7 mm, vias 0 -> 1
- net VPOE: track 56.2 -> 0.00 mm
- net +3V3: track 303.0 -> 301.8 mm
Changed lines of the file:
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@@
 <contactref element="R3" pad="1"/>
 <contactref element="R5" pad="1"/>
-<contactref element="FLOWSENSOR" pad="2"/>
 <contactref element="J5" pad="2"/>
 <contactref element="PRESSURE1" pad="2"/>
@@
 <wire x1="75" y1="49.3645" x2="75" y2="50.5174" width="0.635" layer="1"/>
 <wire x1="75" y1="50.5174" x2="66.8826" y2="50.5174" width="0.635" layer="1"/>
-<wire x1="60.8504" y1="51.7" x2="60.8504" y2="50.1142" width="0.635" layer="1"/>
-<wire x1="66.8826" y1="50.5174" x2="65.7" y2="51.7" width="0.635" layer="1"/>
+<wire x1="66.8826" y1="50.5174" x2="65.3" y2="52.1" width="0.635" layer="1"/>
 <wire x1="75.945" y1="27.755" x2="76" y2="27.7" width="0.254" layer="1"/>
 <wire x1="76" y1="26.7497375" x2="76.6001" y2="26.1496375" width="0.254" layer="1"/>
@@
 <wire x1="63.1" y1="13.4" x2="67.65" y2="8.85" width="0.254" layer="1"/>
 <wire x1="63.1" y1="19.1602" x2="63.1" y2="13.4" width="0.254" layer="1"/>
-<wire x1="60.8504" y1="51.7" x2="50.7" y2="51.7" width="0.635" layer="1"/>
-<wire x1="50.7" y1="51.7" x2="45.8884" y2="46.8884" width="0.635" layer="1"/>
-<wire x1="65.7" y1="51.7" x2="60.8504" y2="51.7" width="0.635" layer="1"/>
+<wire x1="65.3" y1="52.1" x2="51.1" y2="52.1" width="0.635" layer="1"/>
+<wire x1="51.1" y1="52.1" x2="45.8884" y2="46.8884" width="0.635" layer="1"/>
 <wire x1="59.6992" y1="4.7" x2="59.7996" y2="4.8004" width="0.254" layer="1"/>
 <wire x1="46.5991" y1="4.7" x2="42.4742" y2="8.8249" width="0.254" layer="1"/>
 <wire x1="46.5991" y1="4.7" x2="59.6992" y2="4.7" width="0.254" layer="1"/>
 <wire x1="45.8884" y1="46.8884" x2="45.8884" y2="46.7116" width="0.254" layer="1"/>
-<wire x1="51.7" y1="28.5710625" x2="53.6246" y2="26.6464625" width="0.254" layer="1"/>
-<wire x1="45.8884" y1="46.7116" x2="51.7" y2="40.9" width="0.254" layer="1"/>
-<wire x1="51.7" y1="40.9" x2="51.7" y2="28.5710625" width="0.254" layer="1"/>
+<wire x1="50.7" y1="29.5710625" x2="53.6246" y2="26.6464625" width="0.254" layer="1"/>
+<wire x1="45.8884" y1="46.7116" x2="50.7" y2="41.9" width="0.254" layer="1"/>
+<wire x1="50.7" y1="41.9" x2="50.7" y2="29.5710625" width="0.254" layer="1"/>
 <wire x1="53.6246" y1="26.6464625" x2="53.6246" y2="24.13373125" width="0.254" layer="1"/>
 <wire x1="53.6246" y1="24.13373125" x2="53.6246" y2="21.621" width="0.254" layer="1"/>
@@
 <wire x1="11.8872" y1="12.9538" x2="12.605" y2="12.236" width="0.254" layer="1"/>
 </signal>
-<signal name="VPOE">
+<signal name="+5V">
 <contactref element="J1" pad="1"/>
 <wire x1="13.97" y1="6.858" x2="21.2902375" y2="6.858" width="0.762" layer="1"/>
@@
 <wire x1="46" y1="31.7252" x2="46" y2="31.73" width="0.792" layer="1"/>
 <wire x1="46" y1="31.73" x2="48.46" y2="34.19" width="0.792" layer="1"/>
+<contactref element="FLOWSENSOR" pad="2"/>
+<wire x1="48.46" y1="34.19" x2="52.39" y2="34.19" width="0.762" layer="16"/>
+<wire x1="52.39" y1="34.19" x2="52.4" y2="34.2" width="0.762" layer="16"/>
+<via x="52.4" y="34.2" extent="1-16" drill="0.35"/>
+<wire x1="52.4" y1="34.2" x2="52.4" y2="48.5" width="0.254" layer="1"/>
+<wire x1="60.03473125" y1="51.3" x2="60.8504" y2="50.48433125" width="0.254" layer="1"/>
+<wire x1="60.8504" y1="50.48433125" x2="60.8504" y2="50.1142" width="0.254" layer="1"/>
+<wire x1="52.4" y1="48.5" x2="55.2" y2="51.3" width="0.254" layer="1"/>
+<wire x1="55.2" y1="51.3" x2="60.03473125" y2="51.3" width="0.254" layer="1"/>
 </signal>
 <signal name="N$20">
