File: design/pcb/ventmon_t0.3.sch (EAGLE design)
At the start: 74 parts, among them IC1 BME280BM280-HAT, J4 MJ-3536N, J6 Header-16, J7 Header-12, U1 W5500, U2 ADS1115IDGST, Y1 25MHz

Commit message: fixed 5V to flow sensor
Connections:
- removed net VPOE: J1.1, J7.3
- new net +5V: FLOWSENSOR.VCC, J1.1, J7.3
- net +3V3: no longer FLOWSENSOR.VCC
Changed lines of the file:
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@@
 <part name="+3V21" library="supply1" deviceset="+3V3" device="" value="+3V3D"/>
 <part name="FLOWSENSOR" library="SparkFun-Connectors" library_urn="urn:adsk.eagle:library:513" deviceset="QWIIC_CONNECTOR" device="JS-1MM" package3d_urn="urn:adsk.eagle:package:38096/1"/>
-<part name="+3V22" library="supply1" deviceset="+3V3" device="" value="+3V3D"/>
 <part name="U$3" library="microbuilder" deviceset="GND" device=""/>
 <part name="J5" library="SparkFun-Connectors" library_urn="urn:adsk.eagle:library:513" deviceset="QWIIC_CONNECTOR" device="JS-1MM" package3d_urn="urn:adsk.eagle:package:38096/1"/>
@@
 <part name="T1" library="Wurth_Signal &amp; Communications_WE-RJ45_LAN" library_urn="urn:adsk.eagle:library:14284239" deviceset="WE-RJ45_7499210121A" device="" package3d_urn="urn:adsk.eagle:package:12863551/2"/>
 <part name="+3V20" library="supply1" deviceset="+3V3" device="" value="+3V3D"/>
+<part name="P+1" library="supply1" library_urn="urn:adsk.eagle:library:371" deviceset="+5V" device=""/>
 </parts>
 <sheets>
@@
 </segment>
 </net>
-<net name="VPOE" class="0">
+<net name="+5V" class="0">
 <segment>
 <label x="128.27" y="24.384" size="1.778" layer="95"/>
@@
 <attribute name="NAME" x="-33.02" y="-65.786" size="1.778" layer="95" font="vector"/>
 </instance>
-<instance part="+3V22" gate="G$1" x="-7.62" y="-66.04" smashed="yes">
-<attribute name="VALUE" x="-4.064" y="-63.246" size="1.778" layer="96" rot="R180"/>
-</instance>
 <instance part="U$3" gate="G$1" x="-7.62" y="-82.55" smashed="yes">
 <attribute name="VALUE" x="-9.144" y="-85.09" size="1.27" layer="96"/>
@@
 <attribute name="VALUE" x="-78.43" y="72.116" size="1.778" layer="96" font="vector" rot="MR180"/>
 <attribute name="NAME" x="-78.43" y="36.302" size="1.778" layer="95" font="vector" rot="MR180"/>
+</instance>
+<instance part="P+1" gate="1" x="-7.62" y="-63.5" smashed="yes">
+<attribute name="VALUE" x="-7.62" y="-60.96" size="1.778" layer="96" align="top-center"/>
 </instance>
 </instances>
@@
 <pinref part="C19" gate="G$1" pin="P$2"/>
 <junction x="71.12" y="66.04"/>
-</segment>
-<segment>
-<pinref part="FLOWSENSOR" gate="J1" pin="VCC"/>
-<pinref part="+3V22" gate="G$1" pin="+3V3"/>
-<wire x1="-20.32" y1="-73.66" x2="-7.62" y2="-73.66" width="0.1524" layer="91"/>
-<wire x1="-7.62" y1="-73.66" x2="-7.62" y2="-68.58" width="0.1524" layer="91"/>
 </segment>
 <segment>
@@
 </segment>
 </net>
-<net name="VPOE" class="0">
+<net name="+5V" class="0">
 <segment>
 <pinref part="J7" gate="G$1" pin="3"/>
@@
 <label x="-66" y="62.42" size="1.778" layer="95"/>
 </segment>
-</net>
+<segment>
+<pinref part="FLOWSENSOR" gate="J1" pin="VCC"/>
+<wire x1="-20.32" y1="-73.66" x2="-7.62" y2="-73.66" width="0.1524" layer="91"/>
+<wire x1="-7.62" y1="-73.66" x2="-7.62" y2="-66.04" width="0.1524" layer="91"/>
+<pinref part="P+1" gate="1" pin="+5V"/>
+</segment>
+</net>
